File: VCU/VCU.kicad_sch (KiCad schematic)
At the start: 28 parts, among them J1 LEMO6, J2 LEMO4, J3 Conn_01x10_Male, J4 Conn_01x04_Male, J5 Conn_Coaxial, U1 EL2140, U2 LM7808_TO220

Commit message: Modifying VCU PCB
Connections:
- net +12V: now also C4.1, C5.1, C6.1, U2.1 (VI); no longer C7.1, C8.1, U2.3 (VO)
- net +8V: now also C7.1, C8.1, U2.3 (VO); no longer C4.1, C5.1, C6.1, U2.1 (VI)

Commit message: 12V Modifying
Connections:
- net +12V renamed 12V
Changed lines of the file:
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@@
     (comment 1 "THARWAT AGAMY")
   )
+  (junction (at 31.75 142.24) (diameter 0) (color 0 0 0 0)
+  )
   (junction (at 125.73 142.24) (diameter 0) (color 0 0 0 0)
   )
+  (junction (at 130.81 40.64) (diameter 0) (color 0 0 0 0)
+  )
+  (junction (at 137.16 97.79) (diameter 0) (color 0 0 0 0)
+  )
+  (junction (at 49.53 156.21) (diameter 0) (color 0 0 0 0)
+  )
+  (junction (at 49.53 142.24) (diameter 0) (color 0 0 0 0)
+  )
+  (junction (at 77.47 29.21) (diameter 0) (color 0 0 0 0)
+  )
+  (junction (at 146.05 55.88) (diameter 0) (color 0 0 0 0)
+  )
   (junction (at 69.85 156.21) (diameter 0) (color 0 0 0 0)
   )
-  (junction (at 130.81 40.64) (diameter 0) (color 0 0 0 0)
-  )
-  (junction (at 137.16 97.79) (diameter 0) (color 0 0 0 0)
-  )
-  (junction (at 49.53 156.21) (diameter 0) (color 0 0 0 0)
-  )
-  (junction (at 49.53 142.24) (diameter 0) (color 0 0 0 0)
-  )
-  (junction (at 77.47 29.21) (diameter 0) (color 0 0 0 0)
-  )
-  (junction (at 146.05 55.88) (diameter 0) (color 0 0 0 0)
-  )
   (junction (at 88.9 156.21) (diameter 0) (color 0 0 0 0)
   )
@@
   (junction (at 107.95 156.21) (diameter 0) (color 0 0 0 0)
   )
+  (junction (at 69.85 142.24) (diameter 0) (color 0 0 0 0)
+  )
   (junction (at 146.05 40.64) (diameter 0) (color 0 0 0 0)
   )
   (junction (at 102.87 40.64) (diameter 0) (color 0 0 0 0)
   )
-  (junction (at 69.85 142.24) (diameter 0) (color 0 0 0 0)
-  )
   (junction (at 107.95 142.24) (diameter 0) (color 0 0 0 0)
   )
   (junction (at 228.6 137.16) (diameter 0) (color 0 0 0 0)
-  )
-  (junction (at 31.75 142.24) (diameter 0) (color 0 0 0 0)
   )
   (no_connect (at 36.83 101.6))
@@
   (no_connect (at 245.11 90.17))
   (no_connect (at 49.53 83.82))
+  (wire (pts (xy 69.85 142.24) (xy 81.28 142.24))
+    (stroke (width 0) (type default))
+  )
   (polyline (pts (xy 96.52 189.23) (xy 24.13 189.23))
     (stroke (width 0) (type default))
@@
     (stroke (width 0) (type default))
   )
+  (wire (pts (xy 31.75 134.62) (xy 31.75 142.24))
+    (stroke (width 0) (type default))
+  )
+  (wire (pts (xy 193.04 93.98) (xy 193.04 100.33))
+    (stroke (width 0) (type default))
+  )
   (wire (pts (xy 215.9 134.62) (xy 240.03 134.62))
     (stroke (width 0) (type default))
@@
     (stroke (width 0) (type default))
   )
+  (wire (pts (xy 228.6 85.09) (xy 245.11 85.09))
+    (stroke (width 0) (type default))
+  )
+  (wire (pts (xy 49.53 114.3) (xy 49.53 109.22))
+    (stroke (width 0) (type default))
+  )
+  (wire (pts (xy 107.95 156.21) (xy 88.9 156.21))
+    (stroke (width 0) (type default))
+  )
+  (polyline (pts (xy 187.96 77.47) (xy 187.96 118.11))
+    (stroke (width 0) (type default))
+  )
+  (wire (pts (xy 88.9 40.64) (xy 102.87 40.64))
+    (stroke (width 0) (type default))
+  )
+  (wire (pts (xy 125.73 142.24) (xy 107.95 142.24))
+    (stroke (width 0) (type default))
+  )
+  (wire (pts (xy 31.75 142.24) (xy 49.53 142.24))
+    (stroke (width 0) (type default))
+  )
+  (wire (pts (xy 125.73 144.78) (xy 125.73 142.24))
+    (stroke (width 0) (type default))
+  )
+  (polyline (pts (xy 24.13 167.64) (xy 139.7 167.64))
+    (stroke (width 0) (type default))
+  )
+  (wire (pts (xy 130.81 40.64) (xy 146.05 40.64))
+    (stroke (width 0) (type default))
+  )
+  (polyline (pts (xy 260.35 148.59) (xy 187.96 148.59))
+    (stroke (width 0) (type default))
+  )
+  (polyline (pts (xy 180.34 77.47) (xy 180.34 118.11))
+    (stroke (width 0) (type default))
+  )
+  (wire (pts (xy 31.75 152.4) (xy 31.75 156.21))
+    (stroke (width 0) (type default))
+  )
+  (polyline (pts (xy 260.35 68.58) (xy 260.35 16.51))
+    (stroke (width 0) (type default))
+  )
+  (polyline (pts (xy 95.25 118.11) (xy 95.25 77.47))
+    (stroke (width 0) (type default))
+  )
+  (wire (pts (xy 125.73 137.16) (xy 125.73 142.24))
+    (stroke (width 0) (type default))
+  )
+  (wire (pts (xy 146.05 53.34) (xy 146.05 55.88))
+    (stroke (width 0) (type default))
+  )
+  (wire (pts (xy 31.75 144.78) (xy 31.75 142.24))
+    (stroke (width 0) (type default))
+  )
+  (wire (pts (xy 176.53 40.64) (xy 204.47 40.64))
+    (stroke (width 0) (type default))
+  )
+  (polyline (pts (xy 24.13 16.51) (xy 260.35 16.51))
+    (stroke (width 0) (type default))
+  )
   (wire (pts (xy 88.9 156.21) (xy 88.9 160.02))
     (stroke (width 0) (type default))
   )
-  (wire (pts (xy 228.6 85.09) (xy 245.11 85.09))
-    (stroke (width 0) (type default))
-  )
-  (wire (pts (xy 49.53 114.3) (xy 49.53 109.22))
-    (stroke (width 0) (type default))
-  )
-  (wire (pts (xy 107.95 156.21) (xy 88.9 156.21))
-    (stroke (width 0) (type default))
-  )
-  (polyline (pts (xy 187.96 77.47) (xy 187.96 118.11))
-    (stroke (width 0) (type default))
-  )
-  (wire (pts (xy 88.9 40.64) (xy 102.87 40.64))
-    (stroke (width 0) (type default))
-  )
-  (wire (pts (xy 125.73 142.24) (xy 107.95 142.24))
-    (stroke (width 0) (type default))
-  )
-  (wire (pts (xy 31.75 142.24) (xy 49.53 142.24))
-    (stroke (width 0) (type default))
-  )
-  (wire (pts (xy 125.73 144.78) (xy 125.73 142.24))
-    (stroke (width 0) (type default))
-  )
-  (polyline (pts (xy 24.13 167.64) (xy 139.7 167.64))
-    (stroke (width 0) (type default))
-  )
-  (wire (pts (xy 130.81 40.64) (xy 146.05 40.64))
-    (stroke (width 0) (type default))
-  )
-  (polyline (pts (xy 260.35 148.59) (xy 187.96 148.59))
-    (stroke (width 0) (type default))
-  )
-  (polyline (pts (xy 180.34 77.47) (xy 180.34 118.11))
-    (stroke (width 0) (type default))
-  )
-  (wire (pts (xy 31.75 152.4) (xy 31.75 156.21))
-    (stroke (width 0) (type default))
-  )
-  (polyline (pts (xy 260.35 68.58) (xy 260.35 16.51))
-    (stroke (width 0) (type default))
-  )
-  (polyline (pts (xy 95.25 118.11) (xy 95.25 77.47))
-    (stroke (width 0) (type default))
-  )
-  (wire (pts (xy 125.73 137.16) (xy 125.73 142.24))
-    (stroke (width 0) (type default))
-  )
-  (wire (pts (xy 146.05 53.34) (xy 146.05 55.88))
-    (stroke (width 0) (type default))
-  )
-  (wire (pts (xy 31.75 144.78) (xy 31.75 142.24))
-    (stroke (width 0) (type default))
-  )
-  (wire (pts (xy 176.53 40.64) (xy 204.47 40.64))
-    (stroke (width 0) (type default))
-  )
-  (polyline (pts (xy 24.13 16.51) (xy 260.35 16.51))
-    (stroke (width 0) (type default))
-  )
   (wire (pts (xy 167.64 105.41) (xy 173.99 105.41))
     (stroke (width 0) (type default))
@@
     (stroke (width 0) (type default))
   )
-  (wire (pts (xy 81.28 142.24) (xy 69.85 142.24))
-    (stroke (width 0) (type default))
-  )
   (wire (pts (xy 146.05 55.88) (xy 146.05 58.42))
     (stroke (width 0) (type default))
@@
     (stroke (width 0) (type default))
   )
+  (wire (pts (xy 69.85 156.21) (xy 88.9 156.21))
+    (stroke (width 0) (type default))
+  )
   (polyline (pts (xy 24.13 127) (xy 24.13 167.64))
     (stroke (width 0) (type default))
@@
     (stroke (width 0) (type default))
   )
-  (wire (pts (xy 88.9 156.21) (xy 69.85 156.21))
-    (stroke (width 0) (type default))
-  )
   (wire (pts (xy 31.75 179.07) (xy 53.34 179.07))
     (stroke (width 0) (type default))
@@
   )
   (wire (pts (xy 146.05 40.64) (xy 146.05 45.72))
-    (stroke (width 0) (type default))
-  )
-  (wire (pts (xy 31.75 137.16) (xy 31.75 142.24))
-    (stroke (width 0) (type default))
-  )
-  (wire (pts (xy 193.04 97.79) (xy 193.04 100.33))
     (stroke (width 0) (type default))
   )
@@
   (text "SINGLE SUPPLY TWISTED PAIR DRIVER" (at 24.13 72.39 0)
     (effects (font (size 2 2)) (justify left bottom))
+  )
+  (global_label "12V" (shape input) (at 31.75 134.62 90) (fields_autoplaced)
+    (effects (font (size 1.27 1.27)) (justify left))
+    (property "Intersheetrefs" "${INTERSHEET_REFS}" (at 31.75 128.1272 90)
+      (effects (font (size 1.27 1.27)) (justify left) hide)
+    )
+  )
+  (global_label "12V" (shape output) (at 193.04 93.98 90) (fields_autoplaced)
+    (effects (font (size 1.27 1.27)) (justify left))
+    (property "Intersheetrefs" "${INTERSHEET_REFS}" (at 193.04 87.4872 90)
+      (effects (font (size 1.27 1.27)) (justify left) hide)
+    )
   )
   (hierarchical_label "Video_2_to_J5" (shape output) (at 215.9 139.7 180) (fields_autoplaced)
@@
     )
   )
-  (symbol (lib_id "power:+12V") (at 31.75 137.16 0) (unit 1)
-    (in_bom yes) (on_board yes) (dnp no)
-    (property "Reference" "#PWR01" (at 31.75 140.97 0)
-      (effects (font (size 1.27 1.27)) hide)
-    )
-    (property "Value" "+12V" (at 31.75 133.35 0)
-      (effects (font (size 1.27 1.27)))
-    )
-    (property "Footprint" "" (at 31.75 137.16 0)
-      (effects (font (size 1.27 1.27)) hide)
-    )
-    (property "Datasheet" "" (at 31.75 137.16 0)
-      (effects (font (size 1.27 1.27)) hide)
-    )
-    (pin "1")
-    (instances
-      (project "VCU"
-        (path "/e782347d-c585-48ee-a745-02943601cb93"
-          (reference "#PWR01") (unit 1)
-        )
-      )
-    )
-  )
   (symbol (lib_id "power:GND") (at 186.69 33.02 0) (unit 1)
     (in_bom yes) (on_board yes) (dnp no)
@@
         )
       )
-    )
-  )
-  (symbol (lib_id "power:+12V") (at 193.04 97.79 0) (unit 1)
-    (in_bom yes) (on_board yes) (dnp no) (fields_autoplaced)
-    (property "Reference" "#PWR0103" (at 193.04 101.6 0)
-      (effects (font (size 1.27 1.27)) hide)
-    )
-    (property "Value" "+12V" (at 193.04 92.71 0)
-      (effects (font (size 1.27 1.27)))
-    )
-    (property "Footprint" "" (at 193.04 97.79 0)
-      (effects (font (size 1.27 1.27)) hide)
-    )
-    (property "Datasheet" "" (at 193.04 97.79 0)
-      (effects (font (size 1.27 1.27)) hide)
-    )
-    (pin "1")
-    (instances
-      (project "VCU"
-        (path "/e782347d-c585-48ee-a745-02943601cb93"
-          (reference "#PWR0103") (unit 1)
-        )
-      )
